Commit message: update : urdf

File: rider_description/urdf/rider_basic.urdf (robot description, URDF)
Before this commit: robot rider_description, 8 links, 7 joints
Joints:
- removed joint joint_name
- added joint caster_joint: type fixed, parent base_link, child caster_link, origin xyz=-0.081 0.0 -0.004 rpy=0.0 0.0 0.0
